Commit message: rough urdf model, robot state publisher

File: description/robot.urdf.xacro (robot description, xacro)
@@ -2,4 +2,3 @@
 <robot xmlns:xacro="http://www.ros.org/wiki/xacro"  name="my_robot">
         <xacro:include filename="robot_core.xacro" />
-        <xacro:include filename="gazebo_control.xacro"/>
 </robot>

File: description/robot_core.xacro (robot description, xacro)
@@ -1,142 +1,150 @@
 <?xml version="1.0"?>
 <robot xmlns:xacro="http://www.ros.org/wiki/xacro" >
-    <xacro:include filename="inertial_macros.xacro"/>
-    <xacro:property name="chassis_length" value="0.335"/>
-    <xacro:property name="chassis_width" value="0.265"/>
-    <xacro:property name="chassis_height" value="0.138"/>
-    <xacro:property name="chassis_mass" value="1.0"/>
-    <xacro:property name="wheel_radius" value="0.033"/>
-    <xacro:property name="wheel_thickness" value="0.026"/>
-    <xacro:property name="wheel_mass" value="0.05"/>
-    <xacro:property name="wheel_offset_x" value="0.226"/>
-    <xacro:property name="wheel_offset_y" value="0.1485"/>
-    <xacro:property name="wheel_offset_z" value="0.01"/>
-    <xacro:property name="caster_wheel_radius" value="0.01"/>
-    <xacro:property name="caster_wheel_mass" value="0.01"/>
-    <xacro:property name="caster_wheel_offset_x" value="0.075"/>
-    <xacro:property name="caster_wheel_offset_z" value="${wheel_offset_z - wheel_radius + caster_wheel_radius}"/>
-    <material name="white">
-        <color rgba="1 1 1 1" />
-    </material>
-    <material name="orange">
-        <color rgba="1 0.3 0.1 1"/>
-    </material>
-    <material name="blue">
-        <color rgba="0.2 0.2 1 1"/>
-    </material>
-    <material name="black">
-        <color rgba="0 0 0 1"/>
-    </material>
-    <material name="red">
-        <color rgba="1 0 0 1"/>
-    </material>
-    <!-- BASE LINK -->
-    <link name="base_link">
-    </link>
-    <!-- CHASSIS LINK -->
-    <joint name="chassis_joint" type="fixed">
-        <parent link="base_link"/>
-        <child link="chassis"/>
-        <origin xyz="${-wheel_offset_x} 0 ${-wheel_offset_z}"/>
-    </joint>
-    <link name="chassis">
-        <visual>
-            <origin xyz="${chassis_length/2} 0 ${chassis_height/2}"/>
-            <geometry>
-                <box size="${chassis_length} ${chassis_width} ${chassis_height}"/>
-            </geometry>
-            <material name="orange"/>
-        </visual>
-        <collision>
-            <origin xyz="${chassis_length/2} 0 ${chassis_height/2}"/>
-            <geometry>
-                <box size="${chassis_length} ${chassis_width} ${chassis_height}"/>
-            </geometry>
-        </collision>
-        <xacro:inertial_box mass="0.5" x="${chassis_length}" y="${chassis_width}" z="${chassis_height}">
-            <origin xyz="${chassis_length/2} 0 ${chassis_height/2}" rpy="0 0 0"/>
-        </xacro:inertial_box>
-    </link>
-    <gazebo reference="chassis">
-        <material>Gazebo/Orange</material>
-    </gazebo>
-    <!-- LEFT WHEEL LINK -->
-    <joint name="left_wheel_joint" type="continuous">
-        <parent link="base_link"/>
-        <child link="left_wheel"/>
-        <origin xyz="0 ${wheel_offset_y} 0" rpy="-${pi/2} 0 0" />
-        <axis xyz="0 0 1"/>
-    </joint>
-    <link name="left_wheel">
-        <visual>
-            <geometry>
-                <cylinder radius="${wheel_radius}" length="${wheel_thickness}"/>
-            </geometry>
-            <material name="blue"/>
-        </visual>
-        <collision>
-            <geometry>
-                <sphere radius="${wheel_radius}"/>
-            </geometry>
-        </collision>
-        <xacro:inertial_cylinder mass="${wheel_mass}" length="${wheel_thickness}" radius="${wheel_radius}">
-            <origin xyz="0 0 0" rpy="0 0 0"/>
-        </xacro:inertial_cylinder>
-    </link>
-    <gazebo reference="left_wheel">
-        <material>Gazebo/Blue</material>
-    </gazebo>
-    <!-- RIGHT WHEEL LINK -->
-    <joint name="right_wheel_joint" type="continuous">
-        <parent link="base_link"/>
-        <child link="right_wheel"/>
-        <origin xyz="0 ${-wheel_offset_y} 0" rpy="${pi/2} 0 0" />
-        <axis xyz="0 0 -1"/>
-    </joint>
-    <link name="right_wheel">
-        <visual>
-            <geometry>
-                <cylinder radius="${wheel_radius}" length="${wheel_thickness}"/>
-            </geometry>
-            <material name="blue"/>
-        </visual>
-        <collision>
-            <geometry>
-                <sphere radius="${wheel_radius}"/>
-            </geometry>
-        </collision>
-        <xacro:inertial_cylinder mass="${wheel_mass}" length="${wheel_thickness}" radius="${wheel_radius}">
-            <origin xyz="0 0 0" rpy="0 0 0"/>
-        </xacro:inertial_cylinder>
-    </link>
-    <gazebo reference="right_wheel">
-        <material>Gazebo/Blue</material>
-    </gazebo>
-    <!-- CASTER WHEEL LINK -->
-    <joint name="caster_wheel_joint" type="fixed">
-        <parent link="chassis"/>
-        <child link="caster_wheel"/>
-        <origin xyz="${caster_wheel_offset_x} 0 ${caster_wheel_offset_z}"/>
-    </joint>
-    <link name="caster_wheel">
-        <visual>
-            <geometry>
-                <sphere radius="${caster_wheel_radius}"/>
-            </geometry>
-            <material name="white"/>
-        </visual>
-        <collision>
-            <geometry>
-                <sphere radius="${caster_wheel_radius}"/>
-            </geometry>
-        </collision>
-        <xacro:inertial_sphere mass="${caster_wheel_mass}" radius="${caster_wheel_radius}">
-            <origin xyz="0 0 0" rpy="0 0 0"/>
-        </xacro:inertial_sphere>
-    </link>
-    <gazebo reference="caster_wheel">
-        <material>Gazebo/White</material>
-        <mu1 value="0.001"/>
-        <mu2 value="0.001"/>
-    </gazebo>
+	<xacro:include filename="inertial_macros.xacro"/>
+	<xacro:property name="chassis_length" value="0.335"/>
+	<xacro:property name="chassis_width" value="0.265"/>
+	<xacro:property name="chassis_height" value="0.138"/>
+	<xacro:property name="chassis_mass" value="1.0"/>
+	<xacro:property name="wheel_radius" value="0.033"/>
+	<xacro:property name="wheel_thickness" value="0.026"/>
+	<xacro:property name="wheel_mass" value="0.05"/>
+	<xacro:property name="wheel_offset_x" value="0.226"/>
+	<xacro:property name="wheel_offset_y" value="0.1485"/>
+	<xacro:property name="wheel_offset_z" value="0.01"/>
+	<xacro:property name="caster_wheel_radius" value="0.03"/>
+	<xacro:property name="caster_wheel_mass" value="0.03"/>
+	<xacro:property name="caster_wheel_offset_x" value="0.075"/>
+	<xacro:property name="caster_wheel_offset_z" value="${wheel_offset_z - wheel_radius + caster_wheel_radius}"/>
+	<material name="white">
+		<color rgba="1 1 1 1" />
+	</material>
+	<material name="orange">
+		<color rgba="1 0.3 0.1 1"/>
+	</material>
+	<material name="blue">
+		<color rgba="0.2 0.2 1 1"/>
+	</material>
+	<material name="black">
+		<color rgba="0 0 0 1"/>
+	</material>
+	<material name="red">
+		<color rgba="1 0 0 1"/>
+	</material>
+	<!-- BASE LINK -->
+	<link name="base_link">
+	</link>
+	<!-- BASE_FOOTPRINT LINK -->
+	<joint name="base_footprint_joint" type="fixed">
+		<parent link="base_link"/>
+		<child link="base_footprint"/>
+		<origin xyz="0 0 0" rpy="0 0 0"/>
+	</joint>
+	<link name="base_footprint">
+	</link>
+	<!-- CHASSIS LINK -->
+	<joint name="chassis_joint" type="fixed">
+		<parent link="base_link"/>
+		<child link="chassis"/>
+		<origin xyz="${-wheel_offset_x} 0 ${-wheel_offset_z}"/>
+	</joint>
+	<link name="chassis">
+		<visual>
+		<origin xyz="${chassis_length/2} 0 ${chassis_height/2}"/>
+		<geometry>
+			<box size="${chassis_length} ${chassis_width} ${chassis_height}"/>
+		</geometry>
+		<material name="orange"/>
+		</visual>
+		<collision>
+		<origin xyz="${chassis_length/2} 0 ${chassis_height/2}"/>
+		<geometry>
+			<box size="${chassis_length} ${chassis_width} ${chassis_height}"/>
+		</geometry>
+		</collision>
+		<xacro:inertial_box mass="0.5" x="${chassis_length}" y="${chassis_width}" z="${chassis_height}">
+		<origin xyz="${chassis_length/2} 0 ${chassis_height/2}" rpy="0 0 0"/>
+		</xacro:inertial_box>
+	</link>
+	<gazebo reference="chassis">
+		<material>Gazebo/Orange</material>
+	</gazebo>
+	<!-- LEFT WHEEL LINK -->
+	<joint name="left_wheel_joint" type="continuous">
+		<parent link="base_link"/>
+		<child link="left_wheel"/>
+		<origin xyz="0 ${wheel_offset_y} 0" rpy="-${pi/2} 0 0" />
+		<axis xyz="0 0 1"/>
+	</joint>
+	<link name="left_wheel">
+		<visual>
+		<geometry>
+			<cylinder radius="${wheel_radius}" length="${wheel_thickness}"/>
+		</geometry>
+		<material name="blue"/>
+		</visual>
+		<collision>
+		<geometry>
+			<sphere radius="${wheel_radius}"/>
+		</geometry>
+		</collision>
+		<xacro:inertial_cylinder mass="${wheel_mass}" length="${wheel_thickness}" radius="${wheel_radius}">
+		<origin xyz="0 0 0" rpy="0 0 0"/>
+		</xacro:inertial_cylinder>
+	</link>
+	<gazebo reference="left_wheel">
+		<material>Gazebo/Blue</material>
+	</gazebo>
+	<!-- RIGHT WHEEL LINK -->
+	<joint name="right_wheel_joint" type="continuous">
+		<parent link="base_link"/>
+		<child link="right_wheel"/>
+		<origin xyz="0 ${-wheel_offset_y} 0" rpy="${pi/2} 0 0" />
+		<axis xyz="0 0 -1"/>
+	</joint>
+	<link name="right_wheel">
+		<visual>
+		<geometry>
+			<cylinder radius="${wheel_radius}" length="${wheel_thickness}"/>
+		</geometry>
+		<material name="blue"/>
+		</visual>
+		<collision>
+		<geometry>
+			<sphere radius="${wheel_radius}"/>
+		</geometry>
+		</collision>
+		<xacro:inertial_cylinder mass="${wheel_mass}" length="${wheel_thickness}" radius="${wheel_radius}">
+		<origin xyz="0 0 0" rpy="0 0 0"/>
+		</xacro:inertial_cylinder>
+	</link>
+	<gazebo reference="right_wheel">
+		<material>Gazebo/Blue</material>
+	</gazebo>
+	<!-- CASTER WHEEL LINK -->
+	<joint name="caster_wheel_joint" type="fixed">
+		<parent link="chassis"/>
+		<child link="caster_wheel"/>
+		<origin xyz="${caster_wheel_offset_x} 0 ${caster_wheel_offset_z}"/>
+	</joint>
+	<link name="caster_wheel">
+		<visual>
+		<geometry>
+			<sphere radius="${caster_wheel_radius}"/>
+		</geometry>
+		<material name="white"/>
+		</visual>
+		<collision>
+		<geometry>
+			<sphere radius="${caster_wheel_radius}"/>
+		</geometry>
+		</collision>
+		<xacro:inertial_sphere mass="${caster_wheel_mass}" radius="${caster_wheel_radius}">
+		<origin xyz="0 0 0" rpy="0 0 0"/>
+		</xacro:inertial_sphere>
+	</link>
+	<gazebo reference="caster_wheel">
+		<material>Gazebo/White</material>
+		<mu1 value="0.001"/>
+		<mu2 value="0.001"/>
+	</gazebo>
 </robot>

Commit message: move model in urdf, launch file for gazebo

File: description/robot.urdf.xacro (robot description, xacro)
@@ -1,4 +1,5 @@
 <?xml version="1.0"?>
 <robot xmlns:xacro="http://www.ros.org/wiki/xacro"  name="my_robot">
-        <xacro:include filename="robot_core.xacro" />
+        <xacro:include filename="robot_core.xacro"/>
+        <xacro:include filename="gazebo_plugin.xacro"/>
 </robot>

File: description/robot_core.xacro (robot description, xacro)
@@ -1,33 +1,34 @@
 <?xml version="1.0"?>
-<robot xmlns:xacro="http://www.ros.org/wiki/xacro" >
-	<xacro:include filename="inertial_macros.xacro"/>
-	<xacro:property name="chassis_length" value="0.335"/>
-	<xacro:property name="chassis_width" value="0.265"/>
-	<xacro:property name="chassis_height" value="0.138"/>
-	<xacro:property name="chassis_mass" value="1.0"/>
-	<xacro:property name="wheel_radius" value="0.033"/>
-	<xacro:property name="wheel_thickness" value="0.026"/>
-	<xacro:property name="wheel_mass" value="0.05"/>
-	<xacro:property name="wheel_offset_x" value="0.226"/>
-	<xacro:property name="wheel_offset_y" value="0.1485"/>
-	<xacro:property name="wheel_offset_z" value="0.01"/>
-	<xacro:property name="caster_wheel_radius" value="0.03"/>
-	<xacro:property name="caster_wheel_mass" value="0.03"/>
-	<xacro:property name="caster_wheel_offset_x" value="0.075"/>
-	<xacro:property name="caster_wheel_offset_z" value="${wheel_offset_z - wheel_radius + caster_wheel_radius}"/>
+<robot xmlns:xacro="http://www.ros.org/wiki/xacro">
+	<xacro:include filename="inertial_macros.xacro" />
+	<xacro:property name="chassis_length" value="0.35" />
+	<xacro:property name="chassis_width" value="0.3" />
+	<xacro:property name="chassis_height" value="0.15" />
+	<xacro:property name="chassis_mass" value="1.0" />
+	<xacro:property name="wheel_radius" value="0.035" />
+	<xacro:property name="wheel_thickness" value="0.025" />
+	<xacro:property name="wheel_mass" value="0.05" />
+	<xacro:property name="wheel_offset_x" value="0.27" />
+	<xacro:property name="wheel_offset_y" value="${chassis_width / 2 + wheel_thickness / 2}" />
+	<xacro:property name="wheel_offset_z" value="0.01" />
+	<xacro:property name="caster_wheel_radius" value="0.03" />
+	<xacro:property name="caster_wheel_mass" value="0.03" />
+	<xacro:property name="caster_wheel_offset_x" value="0.075" />
+	<xacro:property name="caster_wheel_offset_z"
+		value="${wheel_offset_z - wheel_radius + caster_wheel_radius}" />
 	<material name="white">
 		<color rgba="1 1 1 1" />
 	</material>
 	<material name="orange">
-		<color rgba="1 0.3 0.1 1"/>
+		<color rgba="1 0.3 0.1 1" />
 	</material>
 	<material name="blue">
-		<color rgba="0.2 0.2 1 1"/>
+		<color rgba="0.2 0.2 1 1" />
 	</material>
 	<material name="black">
-		<color rgba="0 0 0 1"/>
+		<color rgba="0 0 0 1" />
 	</material>
 	<material name="red">
-		<color rgba="1 0 0 1"/>
+		<color rgba="1 0 0 1" />
 	</material>
 	<!-- BASE LINK -->
@@ -36,7 +37,7 @@
 	<!-- BASE_FOOTPRINT LINK -->
 	<joint name="base_footprint_joint" type="fixed">
-		<parent link="base_link"/>
-		<child link="base_footprint"/>
-		<origin xyz="0 0 0" rpy="0 0 0"/>
+		<parent link="base_link" />
+		<child link="base_footprint" />
+		<origin xyz="0 0 0" rpy="0 0 0" />
 	</joint>
 	<link name="base_footprint">
@@ -44,24 +45,25 @@
 	<!-- CHASSIS LINK -->
 	<joint name="chassis_joint" type="fixed">
-		<parent link="base_link"/>
-		<child link="chassis"/>
-		<origin xyz="${-wheel_offset_x} 0 ${-wheel_offset_z}"/>
+		<parent link="base_link" />
+		<child link="chassis" />
+		<origin xyz="${-wheel_offset_x} 0 ${-wheel_offset_z}" />
 	</joint>
 	<link name="chassis">
 		<visual>
-		<origin xyz="${chassis_length/2} 0 ${chassis_height/2}"/>
-		<geometry>
-			<box size="${chassis_length} ${chassis_width} ${chassis_height}"/>
-		</geometry>
-		<material name="orange"/>
+			<origin xyz="${chassis_length/2} 0 ${chassis_height/2}" />
+			<geometry>
+				<box size="${chassis_length} ${chassis_width} ${chassis_height}" />
+			</geometry>
+			<material name="orange" />
 		</visual>
 		<collision>
-		<origin xyz="${chassis_length/2} 0 ${chassis_height/2}"/>
-		<geometry>
-			<box size="${chassis_length} ${chassis_width} ${chassis_height}"/>
-		</geometry>
+			<origin xyz="${chassis_length/2} 0 ${chassis_height/2}" />
+			<geometry>
+				<box size="${chassis_length} ${chassis_width} ${chassis_height}" />
+			</geometry>
 		</collision>
-		<xacro:inertial_box mass="0.5" x="${chassis_length}" y="${chassis_width}" z="${chassis_height}">
-		<origin xyz="${chassis_length/2} 0 ${chassis_height/2}" rpy="0 0 0"/>
+		<xacro:inertial_box mass="0.5" x="${chassis_length}" y="${chassis_width}"
+			z="${chassis_height}">
+			<origin xyz="${chassis_length/2} 0 ${chassis_height/2}" rpy="0 0 0" />
 		</xacro:inertial_box>
 	</link>
@@ -71,23 +73,24 @@
 	<!-- LEFT WHEEL LINK -->
 	<joint name="left_wheel_joint" type="continuous">
-		<parent link="base_link"/>
-		<child link="left_wheel"/>
+		<parent link="base_link" />
+		<child link="left_wheel" />
 		<origin xyz="0 ${wheel_offset_y} 0" rpy="-${pi/2} 0 0" />
-		<axis xyz="0 0 1"/>
+		<axis xyz="0 0 1" />
 	</joint>
 	<link name="left_wheel">
 		<visual>
-		<geometry>
-			<cylinder radius="${wheel_radius}" length="${wheel_thickness}"/>
-		</geometry>
-		<material name="blue"/>
+			<geometry>
+				<cylinder radius="${wheel_radius}" length="${wheel_thickness}" />
+			</geometry>
+			<material name="blue" />
 		</visual>
 		<collision>
-		<geometry>
-			<sphere radius="${wheel_radius}"/>
-		</geometry>
+			<geometry>
+				<sphere radius="${wheel_radius}" />
+			</geometry>
 		</collision>
-		<xacro:inertial_cylinder mass="${wheel_mass}" length="${wheel_thickness}" radius="${wheel_radius}">
-		<origin xyz="0 0 0" rpy="0 0 0"/>
+		<xacro:inertial_cylinder mass="${wheel_mass}" length="${wheel_thickness}"
+			radius="${wheel_radius}">
+			<origin xyz="0 0 0" rpy="0 0 0" />
 		</xacro:inertial_cylinder>
 	</link>
@@ -97,23 +100,24 @@
 	<!-- RIGHT WHEEL LINK -->
 	<joint name="right_wheel_joint" type="continuous">
-		<parent link="base_link"/>
-		<child link="right_wheel"/>
+		<parent link="base_link" />
+		<child link="right_wheel" />
 		<origin xyz="0 ${-wheel_offset_y} 0" rpy="${pi/2} 0 0" />
-		<axis xyz="0 0 -1"/>
+		<axis xyz="0 0 -1" />
 	</joint>
 	<link name="right_wheel">
 		<visual>
-		<geometry>
-			<cylinder radius="${wheel_radius}" length="${wheel_thickness}"/>
-		</geometry>
-		<material name="blue"/>
+			<geometry>
+				<cylinder radius="${wheel_radius}" length="${wheel_thickness}" />
+			</geometry>
+			<material name="blue" />
 		</visual>
 		<collision>
-		<geometry>
-			<sphere radius="${wheel_radius}"/>
-		</geometry>
+			<geometry>
+				<sphere radius="${wheel_radius}" />
+			</geometry>
 		</collision>
-		<xacro:inertial_cylinder mass="${wheel_mass}" length="${wheel_thickness}" radius="${wheel_radius}">
-		<origin xyz="0 0 0" rpy="0 0 0"/>
+		<xacro:inertial_cylinder mass="${wheel_mass}" length="${wheel_thickness}"
+			radius="${wheel_radius}">
+			<origin xyz="0 0 0" rpy="0 0 0" />
 		</xacro:inertial_cylinder>
 	</link>
@@ -123,28 +127,28 @@
 	<!-- CASTER WHEEL LINK -->
 	<joint name="caster_wheel_joint" type="fixed">
-		<parent link="chassis"/>
-		<child link="caster_wheel"/>
-		<origin xyz="${caster_wheel_offset_x} 0 ${caster_wheel_offset_z}"/>
+		<parent link="chassis" />
+		<child link="caster_wheel" />
+		<origin xyz="${caster_wheel_offset_x} 0 ${caster_wheel_offset_z}" />
 	</joint>
 	<link name="caster_wheel">
 		<visual>
-		<geometry>
-			<sphere radius="${caster_wheel_radius}"/>
-		</geometry>
-		<material name="white"/>
+			<geometry>
+				<sphere radius="${caster_wheel_radius}" />
+			</geometry>
+			<material name="white" />
 		</visual>
 		<collision>
-		<geometry>
-			<sphere radius="${caster_wheel_radius}"/>
-		</geometry>
+			<geometry>
+				<sphere radius="${caster_wheel_radius}" />
+			</geometry>
 		</collision>
 		<xacro:inertial_sphere mass="${caster_wheel_mass}" radius="${caster_wheel_radius}">
-		<origin xyz="0 0 0" rpy="0 0 0"/>
+			<origin xyz="0 0 0" rpy="0 0 0" />
 		</xacro:inertial_sphere>
 	</link>
 	<gazebo reference="caster_wheel">
 		<material>Gazebo/White</material>
-		<mu1 value="0.001"/>
-		<mu2 value="0.001"/>
+		<mu1 value="0.001" />
+		<mu2 value="0.001" />
 	</gazebo>
 </robot>

Commit message: lidar done

File: description/robot.urdf.xacro (robot description, xacro)
@@ -3,3 +3,4 @@
         <xacro:include filename="robot_core.xacro"/>
         <xacro:include filename="gazebo_plugin.xacro"/>
+        <xacro:include filename="lidar.xacro" />
 </robot>

File: description/robot_core.xacro (robot description, xacro)
@@ -5,5 +5,5 @@
 	<xacro:property name="chassis_width" value="0.3" />
 	<xacro:property name="chassis_height" value="0.15" />
-	<xacro:property name="chassis_mass" value="1.0" />
+	<xacro:property name="chassis_mass" value="0.5" />
 	<xacro:property name="wheel_radius" value="0.035" />
 	<xacro:property name="wheel_thickness" value="0.025" />
@@ -63,5 +63,5 @@
 			</geometry>
 		</collision>
-		<xacro:inertial_box mass="0.5" x="${chassis_length}" y="${chassis_width}"
+		<xacro:inertial_box mass="${chassis_mass}" x="${chassis_length}" y="${chassis_width}"
 			z="${chassis_height}">
 			<origin xyz="${chassis_length/2} 0 ${chassis_height/2}" rpy="0 0 0" />
