Commit message: lidar in rviz, launch rviz

File: description/gazebo_plugin.xacro (robot description, xacro)
@@ -66,11 +66,7 @@
                 filename="ignition-gazebo-joint-state-publisher-system"
                 name="ignition::gazebo::systems::JointStatePublisher">
-                </plugin>
-                <plugin
-                filename="ignition-gazebo-pose-publisher-system"
-                name="ignition::gazebo::systems::PosePublisher">
-                        <publish_link_pose>true</publish_link_pose>
-                        <use_pose_vector_msg>true</use_pose_vector_msg>
-                        <publish_sensor_pose>true</publish_sensor_pose>
+                        <topic>joint_states</topic>
+                        <joint_name>left_wheel_joint</joint_name>
+                        <joint_name>right_wheel_joint</joint_name>
                 </plugin>
         </gazebo>

File: description/lidar.xacro (robot description, xacro)
@@ -3,8 +3,8 @@
         <joint name="lidar_joint" type="fixed">
                 <parent link="chassis" />
-                <child link="lidar_link" />
+                <child link="lidar_frame" />
                 <origin xyz="0.13 0 0.15" rpy="0 0 0" />
         </joint>
-        <link name="lidar_link">
+        <link name="lidar_frame">
                 <visual>
                         <geometry>
@@ -22,5 +22,5 @@
                 </xacro:inertial_cylinder>
         </link>
-        <gazebo reference="lidar_link">
+        <gazebo reference="lidar_frame">
                 <material>Gazebo/Black</material>
                 <sensor name="gpu_lidar" type="gpu_lidar">
@@ -42,6 +42,6 @@
                                 </range>
                         </lidar>
-                        <alwaysOn>1</alwaysOn>
                         <visualize>true</visualize>
+                        <gz_frame_id>lidar_frame</gz_frame_id>
                 </sensor>
         </gazebo>
